Commit message: major updates 1

File: robotarmmanip_description/urdf/arduinobot1.urdf.xacro (robot description, xacro)
@@ -1,4 +1,4 @@
 <?xml version="1.0"?>
-<robot xmlns:xacro="https//www.ros.org/wiki/xacro" name='arduinobot'>
+<robot xmlns:xacro="https//www.ros.org/wiki/xacro" name='robotarmmanip'>
     <xacro:property name="PI" value="3.14159"/>
     <xacro:property name="effort" value="30.0"/>

File: robotarmmanip_description/urdf/robotarmmanip.urdf.xacro (robot description, xacro)
@@ -1,29 +1,4 @@
 <?xml version="1.0"?>
-<robot xmlns:xacro="http://www.ros.org/wiki/xacro" name="arduinobot">
-    <xacro:include filename="$(find arduinobot_description)/urdf/arduinobot_gazebo.xacro"/>
-    <xacro:include filename="$(find arduinobot_description)/urdf/arduinobot_ros2_control.xacro"/>
-    <!-- Useful XACRO Variables (Properties) -->
-    <xacro:property name="PI" value="3.14159265359" />
-    <xacro:property name="effort" value="30.0" />
-    <xacro:property name="velocity" value="10.0" />
-    <!-- Useful Macros -->
-    <xacro:macro name="default_inertial" params="mass">
-        <inertial>
-            <origin xyz="0 0 0" rpy="0 0 0"/>
-            <mass value="${mass}" />
-            <inertia ixx="1.0" ixy="0.0" ixz="0.0"
-                     iyy="1.0" iyz="0.0"
-                     izz="1.0" />
-        </inertial>
-    </xacro:macro>
-    <xacro:macro name="default_transmission" params="number">
-        <transmission name="transmission_${number}">
-            <plugin>transmission_interface/SimpleTransmission</plugin>
-            <actuator name="motor_${number}" role="actuator1"/>
-            <joint name="joint_${number}" role="joint1">
-                <mechanical_reduction>1.0</mechanical_reduction>
-            </joint>
-        </transmission>
-    </xacro:macro>
+<robot xmlns:xacro="http://www.ros.org/wiki/xacro">
     <!-- Links -->
     <link name="world"/>
@@ -133,19 +108,4 @@
         </collision>
     </link>
-    <link name="rgb_camera">
-        <xacro:default_inertial mass="0.001"/>
-        <visual>
-            <origin rpy="-1.57 0 -1.57" xyz="-0.1 0.125 0.15"/>
-            <geometry>
-                <mesh filename="package://arduinobot_description/meshes/pi_camera.STL" scale="0.01 0.01 0.01"/>
-            </geometry>
-        </visual>
-        <collision>
-            <origin rpy="-1.57 0 -1.57" xyz="-0.1 0.125 0.15"/>
-            <geometry>
-                <mesh filename="package://arduinobot_description/meshes/pi_camera.STL" scale="0.01 0.01 0.01"/>
-            </geometry>
-        </collision>
-    </link>
     <!-- Joints -->
     <joint name="virtual_joint" type="fixed">
@@ -200,41 +160,4 @@
         <mimic joint="joint_4" multiplier="-1"/>
     </joint>
-    <joint name ="rgb_camera_joint" type="fixed">
-        <parent link="base_link"/>
-        <child link = "rgb_camera"/>
-        <origin xyz="0 0.45 0.2" rpy="0 -0.5 1.57"/>
-    </joint>
-    <!-- <gazebo reference="rgb_camera">
-        <sensor type="camera" name="rgb_camera">
-            <always_on>true</always_on>
-            <update_rate>30.0</update_rate>
-            <camera name="rgb_camera">
-                <horizontal_fov>1.15</horizontal_fov>
-                <vertical_fov>0.71</vertical_fov>
-                <image>
-                    <width>2304</width>
-                    <height>1296</height>
-                    <format>R8G8B8</format>
-                </image>
-                <distortion>
-                    <k1>0.0</k1>
-                    <k2>0.0</k2>
-                    <k3>0.0</k3>
-                    <p1>0.0</p1>
-                    <p2>0.0</p2>
-                    <center>0.5 0.5</center>
-                </distortion>
-            </camera>
-            <plugin name="gazebo_ros_camera" filename="libgazebo_ros_camera.so">
-                <ros>
-                    <remapping>~/image_raw:=image_raw</remapping>
-                    <remapping>~/camera_info:=camera_info</remapping>
-                </ros>
-                <camera_name>rgb_camera</camera_name>
-                <frame_name>rgb_camera</frame_name>
-                <hack_baseline>0.2</hack_baseline>
-            </plugin>
-        </sensor>
-      </gazebo> -->
     <xacro:default_transmission number="1"/>
     <xacro:default_transmission number="2"/>

File: robotarmmanip_description/urdf/robotarmmanip_gazebo.xacro (robot description, xacro)
@@ -1,4 +1,4 @@
 <?xml version="1.0"?>
-<robot xmlns:xacro="http://www.ros.org/wiki/xacro" name="arduinobot">
+<robot xmlns:xacro="http://www.ros.org/wiki/xacro">
     <gazebo>
         <plugin filename="libgazebo_ros2_control.so" name="gazebo_ros2_control">

File: robotarmmanip_description/urdf/robotarmmanip_ros2_control.xacro (robot description, xacro)
@@ -1,5 +1,4 @@
 <?xml version="1.0"?>
-<robot xmlns:xacro="http://www.ros.org/wiki/xacro" name="arduinobot">
-    <xacro:property name="PI" value="3.14159265359" />
+<robot xmlns:xacro="http://www.ros.org/wiki/xacro" >
     <ros2_control name="RobotSystem" type="system">
         <hardware>
