Commit message: update 02

File: robotarmmanip_description/urdf/rgb_camera.urdf.xacro (robot description, xacro)
@@ -6,5 +6,5 @@
             <origin rpy="-1.57 0 -1.57" xyz="-0.1 0.125 0.15"/>
             <geometry>
-                <mesh filename="package://arduinobot_description/meshes/pi_camera.STL" scale="0.01 0.01 0.01"/>
+                <mesh filename="package://robotarmmanip_description/meshes/pi_camera.STL" scale="0.01 0.01 0.01"/>
             </geometry>
         </visual>
@@ -12,5 +12,5 @@
             <origin rpy="-1.57 0 -1.57" xyz="-0.1 0.125 0.15"/>
             <geometry>
-                <mesh filename="package://arduinobot_description/meshes/pi_camera.STL" scale="0.01 0.01 0.01"/>
+                <mesh filename="package://robotarmmanip_description/meshes/pi_camera.STL" scale="0.01 0.01 0.01"/>
             </geometry>
         </collision>
@@ -18,5 +18,5 @@
     </link>
     <!-- joint -->
-    <joint name ="rgb_camera_joint" type="fixed">
+    <joint name ="base_rgb_camera_joint" type="fixed">
         <parent link="base_link"/>
         <child link = "rgb_camera"/>

File: robotarmmanip_description/urdf/robotarmmanip.urdf.xacro (robot description, xacro)
@@ -8,5 +8,5 @@
             <origin rpy="0 0 0" xyz="-0.5 -0.5 0"/>
             <geometry>
-                <mesh filename="package://arduinobot_description/meshes/basement.STL" scale="0.01 0.01 0.01"/>
+                <mesh filename="package://robotarmmanip_description/meshes/basement.STL" scale="0.01 0.01 0.01"/>
             </geometry>
         </visual>
@@ -14,5 +14,5 @@
             <origin rpy="0 0 0" xyz="-0.5 -0.5 0"/>
             <geometry>
-                <mesh filename="package://arduinobot_description/meshes/basement.STL" scale="0.01 0.01 0.01"/>
+                <mesh filename="package://robotarmmanip_description/meshes/basement.STL" scale="0.01 0.01 0.01"/>
             </geometry>
         </collision>
@@ -23,5 +23,5 @@
             <origin rpy="0 0 0" xyz="-0.39 -0.39 -0.56"/>
             <geometry>
-                <mesh filename="package://arduinobot_description/meshes/base_plate.STL" scale="0.01 0.01 0.01"/>
+                <mesh filename="package://robotarmmanip_description/meshes/base_plate.STL" scale="0.01 0.01 0.01"/>
             </geometry>
         </visual>
@@ -29,5 +29,5 @@
             <origin rpy="0 0 0" xyz="-0.39 -0.39 -0.56"/>
             <geometry>
-                <mesh filename="package://arduinobot_description/meshes/base_plate.STL" scale="0.01 0.01 0.01"/>
+                <mesh filename="package://robotarmmanip_description/meshes/base_plate.STL" scale="0.01 0.01 0.01"/>
             </geometry>
         </collision>
@@ -38,5 +38,5 @@
             <origin rpy=" 0 -${PI / 2} ${PI / 2}" xyz="0.19 0.06 -0.08"/>
             <geometry>
-                <mesh filename="package://arduinobot_description/meshes/forward_drive_arm.STL" scale="0.01 0.01 0.01"/>
+                <mesh filename="package://robotarmmanip_description/meshes/forward_drive_arm.STL" scale="0.01 0.01 0.01"/>
             </geometry>
         </visual>
@@ -44,5 +44,5 @@
             <origin rpy=" 0 -${PI / 2} ${PI / 2}" xyz="0.19 0.06 -0.08"/>
             <geometry>
-                <mesh filename="package://arduinobot_description/meshes/forward_drive_arm.STL" scale="0.01 0.01 0.01"/>
+                <mesh filename="package://robotarmmanip_description/meshes/forward_drive_arm.STL" scale="0.01 0.01 0.01"/>
             </geometry>
         </collision>
@@ -53,5 +53,5 @@
             <origin rpy="${PI / 2} 0 ${PI / 2}" xyz="-0.03 -0.4 -0.06"/>
             <geometry>
-                <mesh filename="package://arduinobot_description/meshes/horizontal_arm.STL" scale="0.01 0.01 0.01"/>
+                <mesh filename="package://robotarmmanip_description/meshes/horizontal_arm.STL" scale="0.01 0.01 0.01"/>
             </geometry>
         </visual>
@@ -59,5 +59,5 @@
             <origin rpy="${PI / 2} 0 ${PI / 2}" xyz="-0.03 -0.4 -0.06"/>
             <geometry>
-                <mesh filename="package://arduinobot_description/meshes/horizontal_arm.STL" scale="0.01 0.01 0.01"/>
+                <mesh filename="package://robotarmmanip_description/meshes/horizontal_arm.STL" scale="0.01 0.01 0.01"/>
             </geometry>
         </collision>
@@ -68,5 +68,5 @@
             <origin rpy="0 0 ${PI / 2}" xyz="0 -0.05 -0.15"/>
             <geometry>
-                <mesh filename="package://arduinobot_description/meshes/claw_support.STL" scale="0.01 0.01 0.01"/>
+                <mesh filename="package://robotarmmanip_description/meshes/claw_support.STL" scale="0.01 0.01 0.01"/>
             </geometry>
         </visual>
@@ -74,5 +74,5 @@
             <origin rpy="0 0 ${PI / 2}" xyz="0 -0.05 -0.15"/>
             <geometry>
-                <mesh filename="package://arduinobot_description/meshes/claw_support.STL" scale="0.01 0.01 0.01"/>
+                <mesh filename="package://robotarmmanip_description/meshes/claw_support.STL" scale="0.01 0.01 0.01"/>
             </geometry>
         </collision>
@@ -83,5 +83,5 @@
             <origin rpy="0 0 -${PI / 2}" xyz="-0.1 0.50 -0.1"/>
             <geometry>
-                <mesh filename="package://arduinobot_description/meshes/right_finger.STL" scale="0.01 0.01 0.01"/>
+                <mesh filename="package://robotarmmanip_description/meshes/right_finger.STL" scale="0.01 0.01 0.01"/>
             </geometry>
         </visual>
@@ -89,5 +89,5 @@
             <origin rpy="0 0 -${PI / 2}" xyz="-0.1 0.50 -0.1"/>
             <geometry>
-                <mesh filename="package://arduinobot_description/meshes/right_finger.STL" scale="0.01 0.01 0.01"/>
+                <mesh filename="package://robotarmmanip_description/meshes/right_finger.STL" scale="0.01 0.01 0.01"/>
             </geometry>
         </collision>
@@ -98,5 +98,5 @@
             <origin rpy="0 0 -${PI / 2}" xyz="-0.04 0.50 -0.1"/>
             <geometry>
-                <mesh filename="package://arduinobot_description/meshes/left_finger.STL" scale="0.01 0.01 0.01"/>
+                <mesh filename="package://robotarmmanip_description/meshes/left_finger.STL" scale="0.01 0.01 0.01"/>
             </geometry>
         </visual>
@@ -104,5 +104,5 @@
             <origin rpy="0 0 -${PI / 2}" xyz="-0.04 0.50 -0.1"/>
             <geometry>
-                <mesh filename="package://arduinobot_description/meshes/left_finger.STL" scale="0.01 0.01 0.01"/>
+                <mesh filename="package://robotarmmanip_description/meshes/left_finger.STL" scale="0.01 0.01 0.01"/>
             </geometry>
         </collision>

File: robotarmmanip_description/urdf/robotarmmanip_all.urdf.xacro (robot description, xacro)
@@ -5,3 +5,4 @@
     <xacro:include filename="$(find robotarmmanip_description)/urdf/robotarmmanip_ros2_control.xacro"/> -->
     <xacro:include filename="$(find robotarmmanip_description)/urdf/robotarmmanip.urdf.xacro" />
+    <xacro:include filename="rgb_camera.urdf.xacro"/>
 </robot>
